Commit message: up

File: robot/config/4wd_car_stereo.urdf.xacro (robot description, xacro)
@@ -182,5 +182,5 @@
   <joint name="stereo_left_camera_joint" type="fixed">
     <parent link="camera_link"/> <child link="stereo_left_camera_link"/>
-    <origin xyz="0 0.03 0" rpy="0 0 0"/>
+    <origin xyz="0 0.05 0" rpy="0 0 0"/>
   </joint>
   <link name="stereo_left_camera_optical"/>
@@ -205,5 +205,5 @@
   <joint name="stereo_right_camera_joint" type="fixed">
     <parent link="camera_link"/> <child link="stereo_right_camera_link"/>
-    <origin xyz="0 -0.03 0" rpy="0 0 0"/>
+    <origin xyz="0 -0.05 0" rpy="0 0 0"/>
   </joint>
   <link name="stereo_right_camera_optical"/>
