Commit message: update xacro

File: robot/config/4wd_car.urdf.xacro (robot description, xacro)
@@ -1,18 +1,38 @@
 <?xml version="1.0"?>
 <robot name="n20_sg90_robot" xmlns:xacro="http://www.ros.org/wiki/xacro">
+  <!-- ===================== -->
+  <!-- 1. 物理参数定义 -->
+  <!-- ===================== -->
+  <!-- 轮子半径（米） -->
   <xacro:property name="wheel_radius" value="0.021"/>
+  <!-- 轮子宽度 -->
   <xacro:property name="wheel_width" value="0.018"/>
+  <!-- 前后轮轴距 -->
   <xacro:property name="wheel_base" value="0.14"/>
+  <!-- 左右轮距 -->
   <xacro:property name="track_width" value="0.12"/>
+  <!-- 车体质量 -->
   <xacro:property name="body_mass" value="0.8"/>
+  <!-- ===================== -->
+  <!-- 2. 材质定义 -->
+  <!-- ===================== -->
   <material name="white"><color rgba="1 1 1 1"/></material>
   <material name="black"><color rgba="0.1 0.1 0.1 1"/></material>
   <material name="red"><color rgba="0.8 0 0 1"/></material>
+  <!-- ===================== -->
+  <!-- 3. Base Frame -->
+  <!-- ===================== -->
+  <!-- ROS 语义用地面投影点（Nav2/TF 标准） -->
   <link name="base_footprint"/>
+  <!-- base_footprint → base_link -->
   <joint name="base_joint" type="fixed">
     <parent link="base_footprint"/>
     <child link="base_link"/>
+    <!-- base_link 抬高一个轮子半径 -->
     <origin xyz="0 0 ${wheel_radius}" rpy="0 0 0"/>
   </joint>
+  <!-- ===================== -->
+  <!-- 4. 车体主体 -->
+  <!-- ===================== -->
   <link name="base_link">
     <visual>
@@ -25,41 +45,72 @@
     <inertial>
       <mass value="${body_mass}"/>
-      <inertia ixx="0.001" ixy="0" ixz="0" iyy="0.003" iyz="0" izz="0.003"/>
+      <!-- 简化惯性矩阵（合理即可） -->
+      <inertia ixx="0.001" ixy="0" ixz="0"
+               iyy="0.003" iyz="0"
+               izz="0.003"/>
     </inertial>
   </link>
+  <!-- ===================== -->
+  <!-- 5. 后轮（驱动轮） -->
+  <!-- ===================== -->
   <xacro:macro name="rear_wheel" params="suffix y_reflect">
     <link name="rear_${suffix}_wheel">
       <visual>
-        <origin rpy="${pi/2} 0 0" xyz="0 0 0"/>
-        <geometry><cylinder radius="${wheel_radius}" length="${wheel_width}"/></geometry>
+        <!-- cylinder 默认轴向是 Z，这里旋转到 Y -->
+        <origin rpy="${pi/2} 0 0"/>
+        <geometry>
+          <cylinder radius="${wheel_radius}" length="${wheel_width}"/>
+        </geometry>
         <material name="black"/>
       </visual>
-      <inertial><mass value="0.05"/><inertia ixx="0.0001" ixy="0" ixz="0" iyy="0.0001" iyz="0" izz="0.0001"/></inertial>
+      <inertial>
+        <mass value="0.05"/>
+        <inertia ixx="0.0001" ixy="0" ixz="0"
+                 iyy="0.0001" iyz="0"
+                 izz="0.0001"/>
+      </inertial>
     </link>
+    <!-- 后轮连续旋转（驱动） -->
     <joint name="rear_${suffix}_wheel_joint" type="continuous">
       <parent link="base_link"/>
       <child link="rear_${suffix}_wheel"/>
-      <origin xyz="-${wheel_base/2} ${y_reflect * track_width/2} 0" rpy="0 0 0"/>
+      <origin xyz="-${wheel_base/2} ${y_reflect * track_width/2} 0"/>
+      <!-- 绕 Y 轴转动 -->
       <axis xyz="0 1 0"/>
     </joint>
   </xacro:macro>
+  <!-- ===================== -->
+  <!-- 6. 前轮（转向 + 旋转） -->
+  <!-- ===================== -->
   <xacro:macro name="front_wheel" params="suffix y_reflect">
+    <!-- 转向关节中间 link（Ackermann 必须） -->
     <link name="front_${suffix}_steer_link">
-      <inertial><mass value="0.02"/><inertia ixx="0.00001" ixy="0" ixz="0" iyy="0.00001" iyz="0" izz="0.00001"/></inertial>
+      <inertial>
+        <mass value="0.02"/>
+        <inertia ixx="0.00001" ixy="0" ixz="0"
+                 iyy="0.00001" iyz="0"
+                 izz="0.00001"/>
+      </inertial>
     </link>
+    <!-- 转向关节 -->
     <joint name="front_${suffix}_steer_joint" type="revolute">
       <parent link="base_link"/>
       <child link="front_${suffix}_steer_link"/>
-      <origin xyz="${wheel_base/2} ${y_reflect * track_width/2} 0" rpy="0 0 0"/>
+      <origin xyz="${wheel_base/2} ${y_reflect * track_width/2} 0"/>
       <axis xyz="0 0 1"/>
+      <!-- ±30° -->
       <limit lower="-0.52" upper="0.52" effort="1.0" velocity="2.0"/>
     </joint>
+    <!-- 实际轮子 -->
     <link name="front_${suffix}_wheel">
       <visual>
-        <origin rpy="${pi/2} 0 0" xyz="0 0 0"/>
-        <geometry><cylinder radius="${wheel_radius}" length="${wheel_width}"/></geometry>
+        <origin rpy="${pi/2} 0 0"/>
+        <geometry>
+          <cylinder radius="${wheel_radius}" length="${wheel_width}"/>
+        </geometry>
         <material name="black"/>
       </visual>
     </link>
+    <!-- 轮子旋转 -->
     <joint name="front_${suffix}_wheel_joint" type="continuous">
       <parent link="front_${suffix}_steer_link"/>
@@ -68,8 +119,12 @@
     </joint>
   </xacro:macro>
-  <xacro:rear_wheel suffix="left" y_reflect="1"/>
-  <xacro:rear_wheel suffix="right" y_reflect="-1"/>
-  <xacro:front_wheel suffix="left" y_reflect="1"/>
+  <!-- 实例化四个轮子 -->
+  <xacro:rear_wheel  suffix="left"  y_reflect="1"/>
+  <xacro:rear_wheel  suffix="right" y_reflect="-1"/>
+  <xacro:front_wheel suffix="left"  y_reflect="1"/>
   <xacro:front_wheel suffix="right" y_reflect="-1"/>
+  <!-- ===================== -->
+  <!-- 7. IMU -->
+  <!-- ===================== -->
   <link name="imu_link"/>
   <joint name="imu_joint" type="fixed">
@@ -78,4 +133,7 @@
     <origin xyz="0 0 0.02"/>
   </joint>
+  <!-- ===================== -->
+  <!-- 8. Camera -->
+  <!-- ===================== -->
   <link name="camera_link">
     <visual>
@@ -87,14 +145,21 @@
     <parent link="base_link"/>
     <child link="camera_link"/>
-    <origin xyz="0.08 0 0.05" rpy="0 0 0"/>
-  </joint>
+    <origin xyz="0.08 0 0.05"/>
+  </joint>
+  <!-- ROS 标准 optical frame -->
   <link name="camera_link_optical"/>
   <joint name="camera_optical_joint" type="fixed">
     <parent link="camera_link"/>
     <child link="camera_link_optical"/>
-    <origin xyz="0 0 0" rpy="${-pi/2} 0 ${-pi/2}"/>
-  </joint>
+    <!-- REP-103 -->
+    <origin rpy="${-pi/2} 0 ${-pi/2}"/>
+  </joint>
+  <!-- ===================== -->
+  <!-- 9. Gazebo 插件 -->
+  <!-- ===================== -->
   <gazebo>
-    <plugin filename="gz-sim-ackermann-steering-system" name="gz::sim::systems::AckermannSteering">
+    <!-- Ackermann 转向系统 -->
+    <plugin filename="gz-sim-ackermann-steering-system"
+            name="gz::sim::systems::AckermannSteering">
       <left_joint>front_left_wheel_joint</left_joint>
       <right_joint>front_right_wheel_joint</right_joint>
@@ -110,4 +175,5 @@
       <child_frame_id>base_link</child_frame_id>
     </plugin>
+    <!-- IMU & 传感器系统 -->
     <plugin filename="gz-sim-imu-system" name="gz::sim::systems::Imu"/>
     <plugin filename="gz-sim-sensors-system" name="gz::sim::systems::Sensors">
@@ -115,4 +181,7 @@
     </plugin>
   </gazebo>
+  <!-- ===================== -->
+  <!-- 10. Gazebo IMU 传感器 -->
+  <!-- ===================== -->
   <gazebo reference="imu_link">
     <sensor name="icm20948" type="imu">
@@ -124,4 +193,7 @@
     </sensor>
   </gazebo>
+  <!-- ===================== -->
+  <!-- 11. Gazebo Camera -->
+  <!-- ===================== -->
   <gazebo reference="camera_link">
     <sensor name="imx219" type="camera">
@@ -138,15 +210,8 @@
           <format>R8G8B8</format>
         </image>
-        <clip><near>0.02</near><far>300</far></clip>
-        <distortion>
-          <k1>0.0</k1><k2>0.0</k2><k3>0.0</k3>
-          <p1>0.0</p1><p2>0.0</p2>
-          <center>0.5 0.5</center>
-        </distortion>
-        <noise>
-          <type>gaussian</type>
-          <mean>0.0</mean>
-          <stddev>0.007</stddev>
-        </noise>
+        <clip>
+          <near>0.02</near>
+          <far>300</far>
+        </clip>
       </camera>
     </sensor>

Commit message: fix sim config

File: robot/config/4wd_car.urdf.xacro (robot description, xacro)
@@ -84,5 +84,5 @@
   <!-- ===================== -->
   <xacro:macro name="front_wheel" params="suffix y_reflect">
-    <!-- 转向关节中间 link（Ackermann 必须） -->
+     <!-- 转向关节中间 link（Ackermann 必须） -->
     <link name="front_${suffix}_steer_link">
       <inertial>
@@ -93,5 +93,5 @@
       </inertial>
     </link>
-    <!-- 转向关节 -->
+     <!-- 转向关节 -->
     <joint name="front_${suffix}_steer_joint" type="revolute">
       <parent link="base_link"/>
@@ -99,5 +99,4 @@
       <origin xyz="${wheel_base/2} ${y_reflect * track_width/2} 0"/>
       <axis xyz="0 0 1"/>
-      <!-- ±30° -->
       <limit lower="-0.52" upper="0.52" effort="1.0" velocity="2.0"/>
     </joint>
@@ -111,4 +110,16 @@
         <material name="black"/>
       </visual>
+      <collision>
+        <origin rpy="${pi/2} 0 0"/>
+        <geometry>
+          <cylinder radius="${wheel_radius}" length="${wheel_width}"/>
+        </geometry>
+      </collision>
+      <inertial>
+        <mass value="0.05"/>
+        <inertia ixx="0.0001" ixy="0" ixz="0"
+                 iyy="0.0001" iyz="0"
+                 izz="0.0001"/>
+      </inertial>
     </link>
     <!-- 轮子旋转 -->
@@ -117,4 +128,5 @@
       <child link="front_${suffix}_wheel"/>
       <axis xyz="0 1 0"/>
+      <dynamics damping="0.1" friction="0.1"/>
     </joint>
   </xacro:macro>

Commit message: up

File: robot/config/4wd_car.urdf.xacro (robot description, xacro)
@@ -70,4 +70,11 @@
                  izz="0.0001"/>
       </inertial>
+      <!-- 碰撞 -->
+      <collision>
+        <origin rpy="${pi/2} 0 0"/>
+        <geometry>
+          <cylinder radius="${wheel_radius}" length="${wheel_width}"/>
+        </geometry>
+      </collision>
     </link>
     <!-- 后轮连续旋转（驱动） -->
@@ -127,4 +134,5 @@
       <parent link="front_${suffix}_steer_link"/>
       <child link="front_${suffix}_wheel"/>
+      <origin xyz="0 0 0" rpy="0 0 0"/>
       <axis xyz="0 1 0"/>
       <dynamics damping="0.1" friction="0.1"/>
@@ -183,5 +191,5 @@
       <wheel_radius>${wheel_radius}</wheel_radius>
       <topic>/cmd_vel</topic>
-      <odom_topic>/ekf/odom</odom_topic>
+      <odom_topic>/wheel_odom</odom_topic>
       <frame_id>odom</frame_id>
       <child_frame_id>base_link</child_frame_id>
@@ -192,4 +200,12 @@
       <render_engine>ogre2</render_engine>
     </plugin>
+    <plugin filename="gz-sim-joint-state-publisher-system"
+        name="gz::sim::systems::JointStatePublisher">
+        <topic>/joint_states</topic>
+        <joint_name>front_left_steer_joint</joint_name>
+        <joint_name>front_right_steer_joint</joint_name>
+        <joint_name>rear_left_wheel_joint</joint_name>
+        <joint_name>rear_right_wheel_joint</joint_name>
+    </plugin>
   </gazebo>
   <!-- ===================== -->
@@ -213,6 +229,6 @@
       <update_rate>30</update_rate>
       <visualize>true</visualize>
-      <topic>camera/image_raw</topic>
-      <gz_frame_id>camera_link</gz_frame_id>
+      <topic>/camera/image_raw</topic>
+      <gz_frame_id>camera_link_optical</gz_frame_id>
       <camera>
         <horizontal_fov>1.085</horizontal_fov>
@@ -226,6 +242,24 @@
           <far>300</far>
         </clip>
+        <!-- 畸变参数 -->
+        <distortion>
+          <k1>0.0</k1> <k2>0.0</k2> <p1>0.0</p1> <p2>0.0</p2>
+          <center>0.5 0.5</center>
+        </distortion>
       </camera>
     </sensor>
   </gazebo>
+  <!-- 轮子摩擦力 -->
+  <gazebo reference="front_left_wheel">
+    <mu1>1.0</mu1><mu2>1.0</mu2><kp>1000000.0</kp><kd>1.0</kd>
+  </gazebo>
+  <gazebo reference="front_right_wheel">
+    <mu1>1.0</mu1><mu2>1.0</mu2><kp>1000000.0</kp><kd>1.0</kd>
+  </gazebo>
+  <gazebo reference="rear_left_wheel">
+    <mu1>1.0</mu1><mu2>1.0</mu2><kp>1000000.0</kp><kd>1.0</kd>
+  </gazebo>
+  <gazebo reference="rear_right_wheel">
+    <mu1>1.0</mu1><mu2>1.0</mu2><kp>1000000.0</kp><kd>1.0</kd>
+  </gazebo>
 </robot>

Commit message: up

File: robot/config/4wd_car.urdf.xacro (robot description, xacro)
@@ -17,7 +17,7 @@
   <!-- 2. 材质定义 -->
   <!-- ===================== -->
-  <material name="white"><color rgba="1 1 1 1"/></material>
-  <material name="black"><color rgba="0.1 0.1 0.1 1"/></material>
-  <material name="red"><color rgba="0.8 0 0 1"/></material>
+  <material name="n20_sg90_robot_white"><color rgba="1 1 1 1"/></material>
+  <material name="n20_sg90_robot_black"><color rgba="0.1 0.1 0.1 1"/></material>
+  <material name="n20_sg90_robot_red"><color rgba="0.8 0 0 1"/></material>
   <!-- ===================== -->
   <!-- 3. Base Frame -->
@@ -38,5 +38,5 @@
     <visual>
       <geometry><box size="0.18 0.1 0.04"/></geometry>
-      <material name="white"/>
+      <material name="n20_sg90_robot_white"/>
     </visual>
     <collision>
@@ -62,5 +62,5 @@
           <cylinder radius="${wheel_radius}" length="${wheel_width}"/>
         </geometry>
-        <material name="black"/>
+        <material name="n20_sg90_robot_black"/>
       </visual>
       <inertial>
@@ -115,5 +115,5 @@
           <cylinder radius="${wheel_radius}" length="${wheel_width}"/>
         </geometry>
-        <material name="black"/>
+        <material name="n20_sg90_robot_black"/>
       </visual>
       <collision>
@@ -159,5 +159,5 @@
     <visual>
       <geometry><box size="0.01 0.03 0.03"/></geometry>
-      <material name="red"/>
+      <material name="n20_sg90_robot_red"/>
     </visual>
   </link>
@@ -197,7 +197,7 @@
     <!-- IMU & 传感器系统 -->
     <plugin filename="gz-sim-imu-system" name="gz::sim::systems::Imu"/>
-    <plugin filename="gz-sim-sensors-system" name="gz::sim::systems::Sensors">
+    <!-- <plugin filename="gz-sim-sensors-system" name="gz::sim::systems::Sensors">
       <render_engine>ogre2</render_engine>
-    </plugin>
+    </plugin> -->
     <plugin filename="gz-sim-joint-state-publisher-system"
         name="gz::sim::systems::JointStatePublisher">
@@ -232,5 +232,5 @@
       <gz_frame_id>camera_link_optical</gz_frame_id>
       <camera>
-        <horizontal_fov>1.085</horizontal_fov>
+        <horizontal_fov>1.0733</horizontal_fov>
         <image>
           <width>1280</width>
@@ -242,8 +242,20 @@
           <far>300</far>
         </clip>
-        <!-- 畸变参数 -->
+        <lens>
+          <intrinsics>
+            <fx>1076.44595</fx>
+            <fy>1074.97836</fy>
+            <cx>621.79270</cx>
+            <cy>359.76983</cy>
+            <s>0.0</s>
+          </intrinsics>
+        </lens>
         <distortion>
-          <k1>0.0</k1> <k2>0.0</k2> <p1>0.0</p1> <p2>0.0</p2>
-          <center>0.5 0.5</center>
+          <k1>-0.23732660</k1>
+          <k2>-0.27874955</k2>
+          <p1>-0.00997783</p1>
+          <p2>0.00048385</p2>
+          <k3>0.48486160</k3>
+          <center>0.4857 0.4997</center>
         </distortion>
       </camera>

Commit message: fix sim issuse

File: robot/config/4wd_car.urdf.xacro (robot description, xacro)
@@ -9,5 +9,5 @@
   <xacro:property name="wheel_width" value="0.018"/>
   <!-- 前后轮轴距 -->
-  <xacro:property name="wheel_base" value="0.14"/>
+  <xacro:property name="wheel_base" value="0.097"/>
   <!-- 左右轮距 -->
   <xacro:property name="track_width" value="0.12"/>
@@ -30,5 +30,5 @@
     <child link="base_link"/>
     <!-- base_link 抬高一个轮子半径 -->
-    <origin xyz="0 0 ${wheel_radius}" rpy="0 0 0"/>
+    <origin xyz="0 0 0.021" rpy="0 0 0"/>
   </joint>
   <!-- ===================== -->
@@ -37,9 +37,9 @@
   <link name="base_link">
     <visual>
-      <geometry><box size="0.18 0.1 0.04"/></geometry>
+      <geometry><box size="0.21 0.09 0.065"/></geometry>
       <material name="n20_sg90_robot_white"/>
     </visual>
     <collision>
-      <geometry><box size="0.18 0.1 0.04"/></geometry>
+      <geometry><box size="0.21 0.09 0.065"/></geometry>
     </collision>
     <inertial>
@@ -151,5 +151,5 @@
     <parent link="base_link"/>
     <child link="imu_link"/>
-    <origin xyz="0 0 0.02"/>
+    <origin xyz="0 0 0.03"/>
   </joint>
   <!-- ===================== -->
@@ -158,5 +158,5 @@
   <link name="camera_link">
     <visual>
-      <geometry><box size="0.01 0.03 0.03"/></geometry>
+      <geometry><box size="0.018 0.025 0.025"/></geometry>
       <material name="n20_sg90_robot_red"/>
     </visual>
@@ -165,5 +165,5 @@
     <parent link="base_link"/>
     <child link="camera_link"/>
-    <origin xyz="0.08 0 0.05"/>
+    <origin xyz="0.1 0 0.05" rpy="0 0.1484 0"/>
   </joint>
   <!-- ROS 标准 optical frame -->
@@ -190,4 +190,6 @@
       <wheel_separation>${track_width}</wheel_separation>
       <wheel_radius>${wheel_radius}</wheel_radius>
+      <kingpin_width>${track_width}</kingpin_width>
+      <steering_limit>0.52</steering_limit>
       <topic>/cmd_vel</topic>
       <odom_topic>/wheel_odom</odom_topic>
@@ -245,5 +247,5 @@
       <gz_frame_id>camera_link_optical</gz_frame_id>
       <camera>
-        <horizontal_fov>1.0733</horizontal_fov>
+        <horizontal_fov>1.815</horizontal_fov>
         <image>
           <width>1280</width>

Commit message: up

File: robot/config/4wd_car.urdf.xacro (robot description, xacro)
@@ -37,9 +37,9 @@
   <link name="base_link">
     <visual>
-      <geometry><box size="0.21 0.09 0.065"/></geometry>
+      <geometry><box size="0.21 0.09 0.021"/></geometry>
       <material name="n20_sg90_robot_white"/>
     </visual>
     <collision>
-      <geometry><box size="0.21 0.09 0.065"/></geometry>
+      <geometry><box size="0.21 0.09 0.021"/></geometry>
     </collision>
     <inertial>

Commit message: up

File: robot/config/4wd_car.urdf.xacro (robot description, xacro)
@@ -165,5 +165,5 @@
     <parent link="base_link"/>
     <child link="camera_link"/>
-    <origin xyz="0.1 0 0.05" rpy="0 0.1484 0"/>
+    <origin xyz="0.1 0 0.05" rpy="0 -0.1484 0"/>
   </joint>
   <!-- ROS 标准 optical frame -->
@@ -247,5 +247,5 @@
       <gz_frame_id>camera_link_optical</gz_frame_id>
       <camera>
-        <horizontal_fov>1.815</horizontal_fov>
+        <horizontal_fov>2.2689</horizontal_fov>
         <image>
           <width>1280</width>

Commit message: up

File: robot/config/4wd_car.urdf.xacro (robot description, xacro)
@@ -165,5 +165,5 @@
     <parent link="base_link"/>
     <child link="camera_link"/>
-    <origin xyz="0.1 0 0.05" rpy="0 -0.1484 0"/>
+    <origin xyz="0.1 0 0.05" rpy="0 0.1484 0"/>
   </joint>
   <!-- ROS 标准 optical frame -->

Commit message: fix momo camera height to 15.1cm

File: robot/config/4wd_car.urdf.xacro (robot description, xacro)
@@ -165,5 +165,5 @@
     <parent link="base_link"/>
     <child link="camera_link"/>
-    <origin xyz="0.1 0 0.05" rpy="0 0.1484 0"/>
+    <origin xyz="0.1 0 0.13" rpy="0 0.1484 0"/>
   </joint>
   <!-- ROS 标准 optical frame -->
